File: 5_Finger_PCB/5_Finger_PCB.kicad_sch (KiCad schematic)
At the start: 0 parts

Commit message: Update five finger PCB schematic
Parts:
- added C1: 10uF, symbol Device:C
- added C2, C4: 100nF, symbol Device:C
- added C3: 1uF, symbol Device:C
- added J1: Conn_01x06, symbol Connector_Generic:Conn_01x06
- added J2: USB_C_Receptacle_USB2.0_16P, symbol Connector:USB_C_Receptacle_USB2.0_16P
- added J3: DXL_MOTOR_1, Connector_JST:JST_EH_B3B-EH-A_1x03_P2.50mm_Vertical, symbol Connector_Generic:Conn_01x03
- added J4: DXL_MOTOR_2, Connector_JST:JST_EH_B3B-EH-A_1x03_P2.50mm_Vertical, symbol Connector_Generic:Conn_01x03
- added J5: DXL_MOTOR_3, Connector_JST:JST_EH_B3B-EH-A_1x03_P2.50mm_Vertical, symbol Connector_Generic:Conn_01x03
- added J6: DXL_MOTOR_4, Connector_JST:JST_EH_B3B-EH-A_1x03_P2.50mm_Vertical, symbol Connector_Generic:Conn_01x03
- added J7: DXL_MOTOR_5, Connector_JST:JST_EH_B3B-EH-A_1x03_P2.50mm_Vertical, symbol Connector_Generic:Conn_01x03
- added R1, R10, R2, R8, R9: 10k, symbol Device:R
- added R3, R4: 22, symbol Device:R
- added R5: 499, symbol Device:R
- added R6, R7: 5.1k, symbol Device:R
- added SW1: RESET, symbol Switch:SW_Push
- added SW2: BOOT, symbol Switch:SW_Push
- added U1: ESP32-S3-WROOM-1-N8R8, RF_Module:ESP32-S3-WROOM-1, symbol RF_Module:ESP32-S3-WROOM-1
- added U2: USBLC6-2SC6, Package_TO_SOT_SMD:SOT-23-6, symbol Power_Protection:USBLC6-2SC6
- added U3: 74LVC2G241, symbol 74xGxx:74LVC2G241
Connections:
- new net: J2.A5 (CC1), R6.1
- new net: J2.A6 (D+), J2.B6 (D+), U2.3 (I/O2)
- new net: J2.A7 (D-), J2.B7 (D-), U2.1 (I/O1)
- new net: J2.B5 (CC2), R7.1
- new net: R3.1, U1.13 (USB_D-)
- new net: R4.1, U1.14 (USB_D+)
- new net: R5.1, U1.37 (TXD0)
- new net DXL_DATA: J3.3 (Pin_3), J4.3 (Pin_3), J5.3 (Pin_3), J6.3 (Pin_3), J7.3 (Pin_3), R8.2, U3.2, U3.3
- new net DXL_TX_EN: R10.1, U1.23 (IO21), U3.1, U3.7
- new net DXL_UART_RX: R9.2, U1.11 (IO18), U3.6
- new net DXL_UART_TX: U1.10 (IO17), U3.5
- new net ESP_EN: C3.1, J1.5 (Pin_5), R1.2, U1.3 (EN)
- new net ESP_GPIO0: J1.6 (Pin_6), R2.2, SW2.2, U1.27 (IO0)
- new net GND: C1.2, C2.1, C3.2, C4.2, J1.2 (Pin_2), J2.A1 (GND), J2.A12 (GND), J2.B1 (GND), J2.B12 (GND), J2.SH (SHIELD), J3.1 (Pin_1), J4.1 (Pin_1), J5.1 (Pin_1), J6.1 (Pin_1), J7.1 (Pin_1), R10.2, R6.2, R7.2, SW1.1, SW1.2, SW2.1, U1.1 (GND), U1.40 (GND), U1.41 (GND), U2.2 (GND), U3.4 (GND)
- new net LOGIC_3V3: C1.1, C2.2, C4.1, J1.1 (Pin_1), R1.1, R2.1, R8.1, R9.1, U1.2 (3V3), U3.8 (VCC)
- new net MOTOR_5V: J3.2 (Pin_2), J4.2 (Pin_2), J5.2 (Pin_2), J6.2 (Pin_2), J7.2 (Pin_2)
- new net UART0_RX: J1.4 (Pin_4), U1.36 (RXD0)
- new net UART0_TX: J1.3 (Pin_3), R5.2
- new net USB_D+: R4.2, U2.4 (I/O2)
- new net USB_D-: R3.2, U2.6 (I/O1)
- new net USB_VBUS: J2.A4 (VBUS), J2.A9 (VBUS), J2.B4 (VBUS), J2.B9 (VBUS), U2.5 (VBUS)
- no-connect marks 0 -> 5

Commit message: Update KiCad schematic
Parts:
- added C5, C6, C7, C8, C9: 100nF, symbol Device:C
- added unit 1 of U3
- added unit 2 of U3
Connections:
- net DXL_DATA: now also C5.2, C6.2, C7.2, C8.2, C9.2, U3.2, U3.3; no longer U3.2, U3.3
- net DXL_TX_EN: now also U3.1, U3.7; no longer U3.1, U3.7
- net DXL_UART_RX: now also U3.6; no longer U3.6
- net DXL_UART_TX: now also U3.5; no longer U3.5
- net MOTOR_5V: now also C5.1, C6.1, C7.1, C8.1, C9.1
Other:
- moved on the sheet: J3, J4, J5, J6, J7

Commit message: Update KiCad schematic
Parts:
- added C10, C11: 1uF, symbol Device:C
- added C12: 100uF, symbol Device:C_Polarized
- added C13: 100nF, symbol Device:C
- added C14: 10uF, symbol Device:C
- added C15, C16: 22uF, symbol Device:C
- added F1: 7.5A_TBD, symbol Device:Fuse
- added J8: 3S_BATTERY_INPUT, symbol Connector_Generic:Conn_01x02
- added L1: 3.9uH, symbol Device:L
- added Q1: Q_PMOS_GDS, symbol Transistor_FET:Q_PMOS_GDS
- added R11: 300k, symbol Device:R
- added R12: 100k, symbol Device:R
- added TP1: DXL_DATA TestPoint, symbol Connector:TestPoint
- added TP2: DXL_UART_TX TestPoint, symbol Connector:TestPoint
- added TP3: DXL_UART_RX TestPoint, symbol Connector:TestPoint
- added TP4: DXL_TX_EN TestPoint, symbol Connector:TestPoint
- added TP5: TP_LOGIC_3V3, symbol Connector:TestPoint
- added TP6: TP_MOTOR_5V, symbol Connector:TestPoint
- added TP7: TP_GND, symbol Connector:TestPoint
- added U4: TPS2116DRL, Package_TO_SOT_SMD:SOT-583-8, symbol Power_Management:TPS2116DRL
- added U5: AP63203WU, Package_TO_SOT_SMD:TSOT-23-6, symbol Regulator_Switching:AP63203WU
Connections:
- net DXL_DATA: now also TP1.1
- net DXL_TX_EN: now also TP4.1
- net DXL_UART_RX: now also TP3.1
- net DXL_UART_TX: now also TP2.1
- net GND: now also C10.2, C11.2, C12.2, C14.2, C15.2, C16.2, J8.2 (Pin_2), R12.2, TP7.1, U4.1 (GND), U5.4 (GND)
- net LOGIC_3V3: now also C15.1, C16.1, L1.2, TP5.1, U5.1 (FB)
- net MOTOR_5V: now also TP6.1
- net USB_VBUS: now also C10.1, R11.1, U4.3 (VIN1), U4.5 (MODE)
- new net: C13.1, L1.1, U5.5 (SW)
- new net: C13.2, U5.6 (BST)
- new net: R11.2, R12.1, U4.4 (PR1)
- new net BAT_FUSED: F1.2
- new net BAT_RAW: F1.1, J8.1 (Pin_1)
- new net LOGIC_5V: C12.1, C14.1, U4.2 (VOUT), U4.7 (VOUT), U5.2 (EN), U5.3 (IN)
- new net SYS_5V: C11.1, U4.6 (VIN2)
- no-connect marks 5 -> 6

Commit message: Assign 0805 footprints to passives, testpoints, header connectors, and switches
Parts:
- C1, C10, C11, C13, C14, C2, C3, C4, C5, C6, C7, C8, C9: footprint (none) -> Capacitor_SMD:C_0805_2012Metric
- J1: footprint (none) -> Connector_PinHeader_2.54mm:PinHeader_1x06_P2.54mm_Vertical
- J8: footprint (none) -> Connector_JST:JST_XH_B2B-XH-A_1x02_P2.50mm_Vertical
- R1, R10, R11, R12, R2, R3, R4, R5, R6, R7, R8, R9: footprint (none) -> Resistor_SMD:R_0805_2012Metric
- SW1, SW2: footprint (none) -> Button_Switch_SMD:SW_SPST_TL3342
- TP1, TP2, TP3, TP4, TP5, TP6, TP7: footprint (none) -> TestPoint:TestPoint_THTPad_D1.5mm_Drill0.7mm
Changed lines of the file:
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@@
 			)
 		)
-		(property "Footprint" ""
+		(property "Footprint" "TestPoint:TestPoint_THTPad_D1.5mm_Drill0.7mm"
 			(at 58.42 171.45 0)
 			(hide yes)
@@
 			)
 		)
-		(property "Footprint" ""
+		(property "Footprint" "Capacitor_SMD:C_0805_2012Metric"
 			(at 116.84 32.0548 0)
 			(hide yes)
@@
 			)
 		)
-		(property "Footprint" ""
+		(property "Footprint" "Capacitor_SMD:C_0805_2012Metric"
 			(at 86.36 100.6348 0)
 			(hide yes)
@@
 			)
 		)
-		(property "Footprint" ""
+		(property "Footprint" "Connector_JST:JST_XH_B2B-XH-A_1x02_P2.50mm_Vertical"
 			(at 25.4 213.36 0)
 			(hide yes)
@@
 			)
 		)
-		(property "Footprint" ""
+		(property "Footprint" "Capacitor_SMD:C_0805_2012Metric"
 			(at 62.23 33.3248 0)
 			(hide yes)
@@
 			)
 		)
-		(property "Footprint" ""
+		(property "Footprint" "Resistor_SMD:R_0805_2012Metric"
 			(at 93.98 66.548 90)
 			(hide yes)
@@
 			)
 		)
-		(property "Footprint" ""
+		(property "Footprint" "TestPoint:TestPoint_THTPad_D1.5mm_Drill0.7mm"
 			(at 184.15 20.32 0)
 			(hide yes)
@@
 			)
 		)
-		(property "Footprint" ""
+		(property "Footprint" "Resistor_SMD:R_0805_2012Metric"
 			(at 124.46 112.268 90)
 			(hide yes)
@@
 			)
 		)
-		(property "Footprint" ""
+		(property "Footprint" "Capacitor_SMD:C_0805_2012Metric"
 			(at 142.24 32.0548 0)
 			(hide yes)
@@
 			)
 		)
-		(property "Footprint" ""
+		(property "Footprint" "TestPoint:TestPoint_THTPad_D1.5mm_Drill0.7mm"
 			(at 212.09 20.32 0)
 			(hide yes)
@@
 			)
 		)
-		(property "Footprint" ""
+		(property "Footprint" "Capacitor_SMD:C_0805_2012Metric"
 			(at 161.29 155.2448 0)
 			(hide yes)
@@
 			)
 		)
-		(property "Footprint" ""
+		(property "Footprint" "Button_Switch_SMD:SW_SPST_TL3342"
 			(at 45.72 139.7 0)
 			(hide yes)
@@
 			)
 		)
-		(property "Footprint" ""
+		(property "Footprint" "TestPoint:TestPoint_THTPad_D1.5mm_Drill0.7mm"
 			(at 40.64 171.45 0)
 			(hide yes)
@@
 			)
 		)
-		(property "Footprint" ""
+		(property "Footprint" "Button_Switch_SMD:SW_SPST_TL3342"
 			(at 30.48 142.24 0)
 			(hide yes)
@@
 			)
 		)
-		(property "Footprint" ""
+		(property "Footprint" "Resistor_SMD:R_0805_2012Metric"
 			(at 50.292 96.52 90)
 			(hide yes)
@@
 			)
 		)
-		(property "Footprint" ""
+		(property "Footprint" "Capacitor_SMD:C_0805_2012Metric"
 			(at 83.5152 204.47 0)
 			(hide yes)
@@
 			)
 		)
-		(property "Footprint" ""
+		(property "Footprint" "Resistor_SMD:R_0805_2012Metric"
 			(at 86.36 57.912 90)
 			(hide yes)
@@
 			)
 		)
-		(property "Footprint" ""
+		(property "Footprint" "Capacitor_SMD:C_0805_2012Metric"
 			(at 133.35 155.2448 0)
 			(hide yes)
@@
 			)
 		)
-		(property "Footprint" ""
+		(property "Footprint" "Resistor_SMD:R_0805_2012Metric"
 			(at 59.182 96.52 90)
 			(hide yes)
@@
 			)
 		)
-		(property "Footprint" ""
+		(property "Footprint" "Resistor_SMD:R_0805_2012Metric"
 			(at 137.668 172.72 90)
 			(hide yes)
@@
 			)
 		)
-		(property "Footprint" ""
+		(property "Footprint" "Capacitor_SMD:C_0805_2012Metric"
 			(at 35.56 32.0548 0)
 			(hide yes)
@@
 			)
 		)
-		(property "Footprint" ""
+		(property "Footprint" "Resistor_SMD:R_0805_2012Metric"
 			(at 124.46 178.308 90)
 			(hide yes)
@@
 			)
 		)
-		(property "Footprint" ""
+		(property "Footprint" "Capacitor_SMD:C_0805_2012Metric"
 			(at 34.29 193.3448 0)
 			(hide yes)
@@
 			)
 		)
-		(property "Footprint" ""
+		(property "Footprint" "Resistor_SMD:R_0805_2012Metric"
 			(at 130.302 129.54 90)
 			(hide yes)
@@
 			)
 		)
-		(property "Footprint" ""
+		(property "Footprint" "Capacitor_SMD:C_0805_2012Metric"
 			(at 78.74 89.8652 0)
 			(hide yes)
@@
 			)
 		)
-		(property "Footprint" ""
+		(property "Footprint" "TestPoint:TestPoint_THTPad_D1.5mm_Drill0.7mm"
 			(at 21.59 171.45 0)
 			(hide yes)
@@
 			)
 		)
-		(property "Footprint" ""
+		(property "Footprint" "Capacitor_SMD:C_0805_2012Metric"
 			(at 36.5252 121.92 0)
 			(hide yes)
@@
 			)
 		)
-		(property "Footprint" ""
+		(property "Footprint" "TestPoint:TestPoint_THTPad_D1.5mm_Drill0.7mm"
 			(at 160.02 20.32 0)
 			(hide yes)
@@
 			)
 		)
-		(property "Footprint" ""
+		(property "Footprint" "Resistor_SMD:R_0805_2012Metric"
 			(at 228.6 57.658 90)
 			(hide yes)
@@
 			)
 		)
-		(property "Footprint" ""
+		(property "Footprint" "Resistor_SMD:R_0805_2012Metric"
 			(at 116.332 124.46 90)
 			(hide yes)
@@
 			)
 		)
-		(property "Footprint" ""
+		(property "Footprint" "Capacitor_SMD:C_0805_2012Metric"
 			(at 90.17 32.0548 0)
 			(hide yes)
@@
 			)
 		)
-		(property "Footprint" ""
+		(property "Footprint" "Capacitor_SMD:C_0805_2012Metric"
 			(at 253.6952 128.27 0)
 			(hide yes)
@@
 			)
 		)
-		(property "Footprint" ""
+		(property "Footprint" "TestPoint:TestPoint_THTPad_D1.5mm_Drill0.7mm"
 			(at 241.3 20.32 0)
 			(hide yes)
@@
 			)
 		)
-		(property "Footprint" ""
+		(property "Footprint" "Connector_PinHeader_2.54mm:PinHeader_1x06_P2.54mm_Vertical"
 			(at 181.61 121.92 0)
 			(hide yes)
@@
 			)
 		)
-		(property "Footprint" ""
+		(property "Footprint" "Resistor_SMD:R_0805_2012Metric"
 			(at 108.712 133.35 90)
 			(hide yes)
@@
 			)
 		)
-		(property "Footprint" ""
+		(property "Footprint" "Resistor_SMD:R_0805_2012Metric"
 			(at 237.49 60.198 90)
 			(hide yes)

Commit message: Add power module symbol and footprint
Parts:
- added C17, C18, C19, C20, C21: 100nF, Capacitor_SMD:C_0805_2012Metric, symbol Device:C
- added C22, C23: 470uF 25V, Capacitor_SMD:CP_Elec_10x10.2, symbol Device:C_Polarized
- added D1: BZT52C10-7-F, Diode_SMD:D_SOD-123, symbol Device:D_Zener
- added F2, F3: 10A MINI Blade, Fuse:Fuseholder_Blade_Mini_Keystone_3568, symbol Device:Fuse
- added J10: DXL_MOTOR_7, Connector_JST:JST_EH_B3B-EH-A_1x03_P2.50mm_Vertical, symbol Connector_Generic:Conn_01x03
- added J11: DXL_MOTOR_8, Connector_JST:JST_EH_B3B-EH-A_1x03_P2.50mm_Vertical, symbol Connector_Generic:Conn_01x03
- added J12: DXL_MOTOR_9, Connector_JST:JST_EH_B3B-EH-A_1x03_P2.50mm_Vertical, symbol Connector_Generic:Conn_01x03
- added J13: DXL_MOTOR_10, Connector_JST:JST_EH_B3B-EH-A_1x03_P2.50mm_Vertical, symbol Connector_Generic:Conn_01x03
- added J9: DXL_MOTOR_6, Connector_JST:JST_EH_B3B-EH-A_1x03_P2.50mm_Vertical, symbol Connector_Generic:Conn_01x03
- added Q2: 2N7002, Package_TO_SOT_SMD:SOT-23, symbol Transistor_FET:2N7002
- added R13: 100k, Resistor_SMD:R_0805_2012Metric, symbol Device:R
- added R14: 1.60k 0.1%, Resistor_SMD:R_0805_2012Metric, symbol Device:R
- added R15: 20k, Resistor_SMD:R_0805_2012Metric, symbol Device:R
- added R16, R17: 10k, Resistor_SMD:R_0805_2012Metric, symbol Device:R
- added U6: OKL2-T/20-W12P2-C, SigRobotics_Power:MURATA_OKL2-T-20-W12P2-C_0, symbol OKL2-T_20-W12P2-C:OKL2-T_20-W12P2-C
- C1, C14: footprint Capacitor_SMD:C_0805_2012Metric -> Capacitor_SMD:C_1206_3216Metric
- C12: value 100uF -> 100uF 16V; footprint (none) -> Capacitor_SMD:CP_Elec_6.3x5.8
- C15, C16: footprint (none) -> Capacitor_SMD:C_1206_3216Metric
- F1: value 7.5A_TBD -> 15A MINI Blade; footprint (none) -> Fuse:Fuseholder_Blade_Mini_Keystone_3568; Fuseholder_MPN (none) -> 3568; MPN (none) -> 0297015.U
- J2: value USB_C_Receptacle_USB2.0_16P -> USB4105-GF-A; footprint (none) -> Connector_USB:USB_C_Receptacle_GCT_USB4105-xx-A_16P_TopMnt_Horizontal; MPN (none) -> USB4105-GF-A
- J8: value 3S_BATTERY_INPUT -> XT30PW-M; footprint Connector_JST:JST_XH_B2B-XH-A_1x02_P2.50mm_Vertical -> Connector_AMASS:AMASS_XT30PW-M_1x02_P2.50mm_Horizontal; MPN (none) -> XT30PW-M30.G.Y
- L1: footprint (none) -> Inductor_SMD:L_APV_ANR5040
- Q1: value Q_PMOS_GDS -> DMP4015SK3Q-13; footprint (none) -> Package_TO_SOT_SMD:TO-252-2
- U3: value 74LVC2G241 -> 74LVC2G241DP,125; footprint (none) -> Package_SO:TSSOP-8_3x3mm_P0.65mm; MPN (none) -> 74LVC2G241DP,125
Connections:
- net BAT_FUSED: now also Q1.2 (D)
- net BAT_RAW: now also J8.2 (Pin_2); no longer J8.1 (Pin_1)
- net DXL_DATA: now also J10.3 (Pin_3), J11.3 (Pin_3), J12.3 (Pin_3), J13.3 (Pin_3), J9.3 (Pin_3); no longer C5.2, C6.2, C7.2, C8.2, C9.2
- net GND: now also C5.2, C6.2, C7.2, C8.2, C9.2, J8.1 (Pin_1), C17.2, C18.2, C19.2, C20.2, C21.2, C22.2, C23.2, J10.1 (Pin_1), J11.1 (Pin_1), J12.1 (Pin_1), J13.1 (Pin_1), J9.1 (Pin_1), Q2.2 (S), R13.1, R14.2, U6.4 (GROUND), U6.4-2 (GROUND), U6.8 (-SENSE(GROUND)), U6.8-2 (-SENSE(GROUND)); no longer J8.2 (Pin_2)
- net LOGIC_3V3: now also R16.1, R17.1
- net MOTOR_ENABLE_N: now reaches U1.4 (IO4)
- net MOTOR_ENABLE_N: now also Q2.1 (G), R16.2
- net MOTOR_PGOOD: now reaches U1.5 (IO5)
- net MOTOR_PGOOD: now also R17.2, U6.9 (POWER_GOOD_OUT), U6.9-2 (POWER_GOOD_OUT)
- net at Q1.1 (G): now also D1.2 (A), R13.2
- net VIN: now reaches Q1.3 (S)
- net VIN: now also D1.1 (K), R15.1, U6.2 (VIN), U6.2-2 (VIN)
- net MOTOR_5V renamed MOTOR_5V_A
- net MOTOR_5V_A: now also C22.1, F2.2; no longer TP6.1
- new net: R14.1, U6.6 (TRIM), U6.6-2 (TRIM)
- new net: Q2.3 (D), R15.2, U6.1 (ON/OFF_CONTROL), U6.1-2 (ON/OFF_CONTROL)
- new net: U6.10 (SYNCRONIZATION), U6.10-2 (SYNCRONIZATION)
- new net: U6.3 (SEQUENCE/TRACKING), U6.3-2 (SEQUENCE/TRACKING)
- new net MOTOR_5V_B: C17.1, C18.1, C19.1, C20.1, C21.1, C23.1, F3.2, J10.2 (Pin_2), J11.2 (Pin_2), J12.2 (Pin_2), J13.2 (Pin_2), J9.2 (Pin_2)
- new net VOUT: F2.1, F3.1, TP6.1, U6.5 (VOUT), U6.5-2 (VOUT), U6.7 (+SENSE(VOUT)), U6.7-2 (+SENSE(VOUT))
- no-connect marks 6 -> 8
Other:
- moved on the sheet: C10, C11, C12, C3, J2, R11, R12, R6, R7, SW1, SW2, TP1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

Commit message: Update KiCad project schematic
Parts:
- added C24: 10uF 25V, Capacitor_SMD:C_1206_3216Metric, symbol Device:C
- added C25, C26: 22uF 10V, Capacitor_SMD:C_1206_3216Metric, symbol Device:C
- added C27: 100 nF 50 V, Capacitor_SMD:C_0805_2012Metric, symbol Device:C
- added J14: SENSOR_EXPANSION, Connector_JST:JST_GH_BM10B-GHS-TBT_1x10-1MP_P1.25mm_Vertical, symbol Connector_Generic:Conn_01x10
- added L2: 4.7uH, Inductor_SMD:L_Bourns_SRP5030T, symbol Device:L
- added U7: AP63205WU-7, Package_TO_SOT_SMD:TSOT-23-6, symbol Regulator_Switching:AP63205WU
- C22, C23: footprint Capacitor_SMD:CP_Elec_10x10.2 -> Capacitor_SMD:CP_Elec_10x10.5
Connections:
- net GND: now also C24.2, C25.2, C26.1, J14.1 (Pin_1), U7.4 (GND)
- net LOGIC_3V3: now also J14.2 (Pin_2)
- net LOGIC_5V: now also J14.3 (Pin_3)
- net SYS_5V: now also C25.1, C26.2, L2.2, U7.1 (FB)
- net VIN: now also C24.1, U7.2 (EN), U7.3 (IN)
- net SENSOR_ADC2: now reaches U1.12 (IO8)
- net SENSOR_ADC2: now also J14.7 (Pin_7)
- net SENSOR_GPIO1: now reaches U1.17 (IO9)
- net SENSOR_GPIO1: now also J14.8 (Pin_8)
- net SENSOR_GPIO2: now reaches U1.18 (IO10)
- net SENSOR_GPIO2: now also J14.9 (Pin_9)
- net SENSOR_INT: now reaches U1.24 (IO47)
- net SENSOR_INT: now also J14.10 (Pin_10)
- net SENSOR_ADC1: now reaches U1.38 (IO2)
- net SENSOR_ADC1: now also J14.6 (Pin_6)
- net I2C_SDA: now reaches U1.6 (IO6)
- net I2C_SDA: now also J14.4 (Pin_4)
- net I2C_SCL: now reaches U1.7 (IO7)
- net I2C_SCL: now also J14.5 (Pin_5)
- new net: C27.1, U7.6 (BST)
- new net: C27.2, L2.1, U7.5 (SW)
- no-connect marks 8 -> 24
Other:
- moved on the sheet: C17, C18, C19, C20, C21, J10, J11, J12, J13, J9
